File: PCA9685 Replacement/PCA9685 Replacement.kicad_pcb (KiCad board)
At the start: 2 copper layers, 106 x 129 mm, 68 parts, among them J1 PI_I2C, J10 PI_PWR_CTRL, J2 Motor 1, J3 Motor 2, J4 USB_C_PWR, J5 USB_C_CHG, J6 XT30_BAT, J7 LTC2954, J8 PB, J9 J_PI_POWER, Q1 Dual_NMOS_1, Q2 Q_USB_OR, Q3 Q_BAT_OR, Q4 Q_MAIN, Q5 Q_NMOS_GDS, U1 PCA9685PW, U2 MCP73831-2-OT, U3 DW01A, U4 AP2112K-3.3

Commit message: Add files via upload
Parts:
- removed C12: 47 uF, Capacitor_SMD:C_0805_2012Metric
- removed C13: 0.1 uF, Capacitor_SMD:C_0805_2012Metric
- removed C14: 470 uF, Capacitor_THT:CP_Radial_D6.3mm_P2.50mm
- removed C26, C27: 10 uF, Capacitor_SMD:C_0805_2012Metric
- removed F2: F_PWR, Fuse:Fuse_1206_3216Metric
- removed J_BOOST1: U3V70F5_MODULE, Connector_PinHeader_2.54mm:PinHeader_1x04_P2.54mm_Vertical
- removed Q1: Dual_NMOS_1, Package_TO_SOT_SMD:SOT-23-6
- removed Q4: Q_MAIN, Package_TO_SOT_SMD:SOT-23
- removed Q5: Q_NMOS_GDS, Package_TO_SOT_SMD:SOT-23
- removed R10, R18: 100, Resistor_SMD:R_0805_2012Metric
- removed R11: 1k, Resistor_SMD:R_0805_2012Metric
- removed R12, R13, R14: 100k, Resistor_SMD:R_0805_2012Metric
- removed R19: 10k, Resistor_SMD:R_0805_2012Metric
- removed R6, R7: 5.1k, Resistor_SMD:R_0805_2012Metric
- removed U3: DW01A, Package_TO_SOT_SMD:SOT-23-6
- removed U4: AP2112K-3.3, Package_TO_SOT_SMD:SOT-23-5
- added C28: 470 uF, Capacitor_THT:CP_Radial_D10.0mm_P5.00mm, F.Cu at (171.0, 103.0)
- added C29: 0.1 uF, Capacitor_SMD:C_0805_2012Metric, F.Cu at (115.1, 91.0)
- added C9: 56 nF, Capacitor_SMD:C_0805_2012Metric, F.Cu at (145.5, 71.5)
- added D1: 1N4148, Diode_THT:D_DO-35_SOD27_P7.62mm_Horizontal, F.Cu at (136.0, 67.0)
- added D2: 1N4148, Diode_THT:D_DO-35_SOD27_P7.62mm_Horizontal, F.Cu at (136.0, 62.0)
- added J11: J_PI_PWR, Connector_PinHeader_2.54mm:PinHeader_1x04_P2.54mm_Vertical, F.Cu at (202.5, 79.8)
- added J12: PIR, Connector_PinSocket_2.54mm:PinSocket_1x02_P2.54mm_Vertical, F.Cu at (202.5, 123.5)
- added J15: D24V90F5-A, Connector_PinSocket_2.54mm:PinSocket_1x04_P2.54mm_Vertical, F.Cu at (106.0, 114.9)
- added REF**: MountingHole_2.2mm_M2_DIN965, MountingHole:MountingHole_2.2mm_M2_DIN965, F.Cu at (94.5, 81.9)
- added REF**: MountingHole_2.2mm_M2_DIN965, MountingHole:MountingHole_2.2mm_M2_DIN965, F.Cu at (94.5, 117.5)
- added TP10: TP_M1, TestPoint:TestPoint_THTPad_D2.0mm_Drill1.0mm, F.Cu at (171.5, 56.5)
- added TP11: TP_M2, TestPoint:TestPoint_THTPad_D2.0mm_Drill1.0mm, F.Cu at (192.5, 65.0)
- added TP12: TP_5V_MAIN, TestPoint:TestPoint_THTPad_D2.0mm_Drill1.0mm, F.Cu at (154.5, 85.5)
- added TP13: TP_PWR_KILL, TestPoint:TestPoint_Pad_D1.5mm, F.Cu at (150.0, 104.0)
- added TP14: TP_PWR_INT, TestPoint:TestPoint_Pad_D1.5mm, F.Cu at (150.0, 109.5)
- added TP15: TP_EN, TestPoint:TestPoint_Pad_D1.5mm, F.Cu at (138.0, 93.5)
- added TP16: TP_VCC, TestPoint:TestPoint_THTPad_D2.0mm_Drill1.0mm, F.Cu at (139.0, 64.5)
- added TP17: TP_GND3, TestPoint:TestPoint_THTPad_D2.0mm_Drill1.0mm, F.Cu at (189.0, 101.5)
- added TP18: TP_GND4, TestPoint:TestPoint_THTPad_D2.0mm_Drill1.0mm, F.Cu at (182.5, 77.5)
- added TP19: TP_PCA, TestPoint:TestPoint_THTPad_D2.0mm_Drill1.0mm, F.Cu at (167.5, 64.0)
- added TP20: TP_SCL, TestPoint:TestPoint_Pad_D1.5mm, F.Cu at (192.5, 118.0)
- added TP21: TP_SDA, TestPoint:TestPoint_Pad_D1.5mm, F.Cu at (192.5, 114.0)
- added TP4: TP_Jack, TestPoint:TestPoint_THTPad_D2.0mm_Drill1.0mm, F.Cu at (118.5, 52.0)
- added TP5: TP_GND1, TestPoint:TestPoint_THTPad_D2.0mm_Drill1.0mm, F.Cu at (103.0, 71.5)
- added TP6: TP_PI, TestPoint:TestPoint_THTPad_D2.0mm_Drill1.0mm, F.Cu at (196.5, 105.0)
- added TP7: TP_GND2, TestPoint:TestPoint_THTPad_D2.0mm_Drill1.0mm, F.Cu at (150.0, 99.5)
- added TP8: TP_5V_SRC, TestPoint:TestPoint_THTPad_D2.0mm_Drill1.0mm, F.Cu at (143.5, 81.0)
- added TP9: TP_BAT, TestPoint:TestPoint_THTPad_D2.0mm_Drill1.0mm, F.Cu at (122.0, 96.5)
- added U5: LTC4353IMS-PBF, Package_SO:MSOP-16_3x4.039mm_P0.5mm, F.Cu at (144.8, 64.6)
- C10, C21: value 0.1 uF -> 47 uF; footprint Capacitor_SMD:C_0805_2012Metric -> Capacitor_SMD:C_1206_3216Metric
- C11: value 22 uF -> 0.1 uF
- C16: footprint Capacitor_SMD:C_0805_2012Metric -> Capacitor_SMD:C_1206_3216Metric
- C17, C24, C25: footprint Capacitor_THT:CP_Radial_D6.3mm_P2.50mm -> Capacitor_THT:CP_Radial_D10.0mm_P5.00mm
- C22: value 47 uF -> 0.1 uF
- C23: value 470 uF -> 47 uF; footprint Capacitor_THT:CP_Radial_D6.3mm_P2.50mm -> Capacitor_SMD:C_1206_3216Metric
- C3: value 22 uF -> 470 uF; footprint Capacitor_SMD:C_0805_2012Metric -> Capacitor_THT:CP_Radial_D10.0mm_P5.00mm
- C5: value 22 uF -> 1 uF
- C6: value 0.1 uF -> 56 nF
- F1: value F_PWR -> 6A-7.5A; footprint Fuse:Fuse_1206_3216Metric -> Fuse:Fuse_2920_7451Metric_Pad2.10x5.45mm_HandSolder
- F3: footprint Fuse:Fuse_1206_3216Metric -> Fuse:Fuse_2920_7451Metric_Pad2.10x5.45mm_HandSolder
- J1: footprint Connector_PinHeader_2.54mm:PinHeader_1x04_P2.54mm_Vertical -> Connector_PinSocket_2.54mm:PinSocket_1x04_P2.54mm_Vertical
- J10: value PI_PWR_CTRL -> Lidar; footprint Connector_PinHeader_2.54mm:PinHeader_1x03_P2.54mm_Vertical -> Connector_PinHeader_2.54mm:PinHeader_1x05_P2.54mm_Vertical
- J2, J3: footprint Connector_PinHeader_2.54mm:PinHeader_1x03_P2.54mm_Vertical -> Connector_PinSocket_2.54mm:PinSocket_1x03_P2.54mm_Vertical
- J4: value USB_C_PWR -> Barrel_Jack; footprint Connector_USB:USB_C_Receptacle_GCT_USB4125-xx-x-0190_6P_TopMnt_Horizontal -> Connector_BarrelJack:BarrelJack_CUI_PJ-102AH_Horizontal
- J5: value USB_C_CHG -> Button Kill Switch; footprint Connector_USB:USB_C_Receptacle_GCT_USB4125-xx-x-0190_6P_TopMnt_Horizontal -> Connector_PinSocket_2.54mm:PinSocket_1x02_P2.54mm_Vertical
- J7: value LTC2954 -> LTC2954-2
- J8: value PB -> D24V90F5-B; footprint Connector_PinHeader_1.00mm:PinHeader_1x01_P1.00mm_Vertical -> Connector_PinSocket_2.54mm:PinSocket_1x04_P2.54mm_Vertical
- J9: value J_PI_POWER -> Pi GPIO; footprint Connector_PinHeader_1.00mm:PinHeader_1x02_P1.00mm_Vertical -> Connector_PinSocket_2.54mm:PinSocket_1x02_P2.54mm_Vertical
- Q2: value Q_USB_OR -> Q_NMOS_GDS; footprint Package_TO_SOT_SMD:SOT-23 -> Package_SO:PowerPAK_SO-8_Single
- Q3: value Q_BAT_OR -> Q_NMOS_GDS; footprint Package_TO_SOT_SMD:SOT-23 -> Package_SO:PowerPAK_SO-8_Single
- R16, R17: value 100k -> 10k
- R8: value 5.1k -> 49.9k
- U2: value MCP73831-2-OT -> TPS2421-2DDAR; footprint Package_TO_SOT_SMD:SOT-23-5 -> Package_SO:SOIC-8-1EP_3.9x4.9mm_P1.27mm_EP2.29x3mm
- moved J8 169.9 mm to (98.4, 84.5), turned to 90 degrees
- moved J4 166.0 mm to (106.0, 62.3), turned to -90 degrees
- moved J5 149.8 mm to (132.0, 131.0), turned to -90 degrees
- moved J6 147.3 mm to (106.0, 131.5), turned to 90 degrees
- moved C21 140.4 mm to (111.1, 90.5), turned to -90 degrees
- moved C11 140.1 mm to (113.5, 116.0), turned to 90 degrees
- moved R9 136.9 mm to (129.0, 109.5), turned to 90 degrees
- moved Q2 135.4 mm to (131.2, 52.9)
- moved F1 135.2 mm to (109.5, 52.0)
- moved C10 134.4 mm to (120.5, 115.5), turned to 90 degrees
- moved Q3 130.6 mm to (132.7, 75.1)
- moved C7 129.0 mm to (117.0, 116.0), turned to 90 degrees
- moved C3 128.1 mm to (113.5, 69.0)
- moved C18 127.0 mm to (128.0, 98.0), turned to 180 degrees
- moved C4 126.5 mm to (116.0, 58.5)
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Connections:
- C1 pad 2: /3V3 -> +3.3V_PI
- C10 pad 1: GND -> CELL+
- C10 pad 2: /CELL+ -> GND
- C11 pad 1: GND -> CELL+
- C11 pad 2: /CELL+ -> GND
- C15 pad 1: /5V_SRC -> +5V_SRC
- C16 pad 1: /5V_SRC -> +5V_SRC
- C17 pad 1: /5V_SRC -> +5V_SRC
- C18 pad 1: /5V_SRC -> +5V_SRC
- C2 pad 1: /3V3 -> +3.3V_PI
- C20 pad 1: Net-(J7-PDT) -> GND
- C20 pad 2: GND -> Net-(J7-PDT)
- C21 pad 1: /5V_MAIN -> +5V_BAT
- C22 pad 1: /5V_MAIN -> +5V_MAIN
- C23 pad 1: /5V_MAIN -> +5V_MAIN
- C24 pad 1: /5V_MAIN -> +5V_MAIN
- C25 pad 1: /5V_MAIN -> +5V_MAIN
- C3 pad 1: /5V_USB -> +5V_USB
- C4 pad 1: /5V_USB -> +5V_USB
- C5 pad 1: /CHG_VBUS -> Net-(U2-CT)
- C6 pad 1: /CHG_VBUS -> +5V_USB
- C6 pad 2: GND -> Net-(U5-CPO1)
- C7 pad 1: /CELL+ -> CELL+
- C7 pad 2: /CELL- -> GND
- C8 pad 1: /CELL- -> Net-(J7-PB)
- C8 pad 2: Net-(U3-VCC) -> GND
- F1 pad 1: /PWR_VBUS_RAW -> Net-(F1-Pad1)
- F1 pad 2: /5V_USB -> +5V_USB
- F3 pad 1: /5V_MAIN -> +5V_MAIN
- F3 pad 2: /5V_PI -> Net-(J11-Pin_1)
- J1 pad 1: /3V3 -> +3.3V_PI
- J1 pad 3: I2C_SCL -> I2C_SDA
- J1 pad 4: I2C_SDA -> I2C_SCL
- J10 pad 1: /PWR_INT -> +5V_MAIN
- J10 pad 2: /PWR_KILL -> GND
- J10 pad 3: GND -> I2C_SDA
- J2 pad 2: /5V_MAIN -> +5V_MAIN
- J3 pad 2: /5V_MAIN -> +5V_MAIN
- J6 pad 1: /CELL+ -> GND
- J6 pad 2: /CELL- -> CELL+
- J7 pad 1: /5V_SRC -> +5V_SRC
- J8 pad 1: Net-(J7-PB) -> GND
- J9 pad 1: /5V_PI -> /PWR_INT
- J9 pad 2: GND -> /PWR_KILL
- Q2 pad 1: /5V_SRC -> Net-(Q2-G)
- Q2 pad 2: /5V_SRC -> +5V_SRC
- Q2 pad 3: /5V_USB -> +5V_USB
- Q3 pad 1: (no net) -> Net-(Q3-G)
- Q3 pad 2: (no net) -> +5V_SRC
- Q3 pad 3: (no net) -> +5V_BAT
- R1 pad 1: /3V3 -> +3.3V_PI
- R15 pad 2: /3V3 -> +3.3V_PI
- R16 pad 1: /PWR_KILL -> +3.3V_PI
- R16 pad 2: /5V_SRC -> /PWR_KILL
- R17 pad 2: /5V_SRC -> +5V_SRC
- R2 pad 1: /3V3 -> +3.3V_PI
- R8 pad 1: Net-(J5-CC1) -> Net-(U2-ISET)
- R9 pad 1: Net-(J5-CC2) -> Net-(J5-Pin_2)
- R9 pad 2: GND -> Net-(J7-PB)
- U1 pad 28: /3V3 -> +3.3V_PI
- U2 pad 2: GND -> /SYS_EN
- U2 pad 3: /CELL+ -> +5V_SRC
- U2 pad 4: /CHG_VBUS -> GND
- U2 pad 5: Net-(U2-PROG) -> Net-(U2-ISET)
Routing:
- net GND: track 0.00 -> 951.2 mm, vias 0 -> 22
- net +3.3V_PI: track 0.00 -> 193.5 mm, vias 0 -> 2
- net +5V_MAIN: track 0.00 -> 184.5 mm
- net +5V_SRC: track 0.00 -> 162.4 mm
- net +5V_BAT: track 0.00 -> 148.8 mm, vias 0 -> 2
- net +5V_USB: track 0.00 -> 97.8 mm
- net I2C_SCL: track 0.00 -> 86.9 mm, vias 0 -> 3
- net I2C_SDA: track 0.00 -> 79.7 mm, vias 0 -> 3
- net /PWR_KILL: track 0.00 -> 59.2 mm, vias 0 -> 3
- net /PWR_INT: track 0.00 -> 54.5 mm
- net CELL+: track 0.00 -> 45.0 mm
- net Net-(U1-LED15): track 0.00 -> 42.7 mm, vias 0 -> 2
- net Net-(U1-LED14): track 0.00 -> 26.8 mm
- net Net-(Q2-G): track 0.00 -> 25.6 mm, vias 0 -> 2
- net /SYS_EN: track 0.00 -> 23.7 mm, vias 0 -> 2
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Other:
- board size 106 x 129 mm -> 116.4 x 92 mm
