File: PCA9685 Replacement/PCA9685 Replacement.kicad_sch (KiCad schematic)
At the start: 68 parts, among them J1 PI_I2C, J10 PI_PWR_CTRL, J2 Motor 1, J3 Motor 2, J4 USB_C_PWR, J5 USB_C_CHG, J6 XT30_BAT, J7 LTC2954, J8 PB, J9 J_PI_POWER, Q1 Dual_NMOS_1, Q2 Q_USB_OR, Q3 Q_BAT_OR, Q4 Q_MAIN, Q5 Q_NMOS_GDS, U1 PCA9685PW, U2 MCP73831-2-OT, U3 DW01A, U4 AP2112K-3.3

Commit message: Add files via upload
Parts:
- removed C26, C27: 10 uF, Capacitor_SMD:C_0805_2012Metric, symbol Device:C_Small
- removed F2: F_PWR, Fuse:Fuse_1206_3216Metric, symbol Device:Fuse
- removed J10: PI_PWR_CTRL, Connector_PinHeader_2.54mm:PinHeader_1x03_P2.54mm_Vertical, symbol Connector_Generic:Conn_01x03
- removed J4: USB_C_PWR, Connector_USB:USB_C_Receptacle_GCT_USB4125-xx-x-0190_6P_TopMnt_Horizontal, symbol Connector:USB_C_Receptacle_PowerOnly_6P
- removed J5: USB_C_CHG, Connector_USB:USB_C_Receptacle_GCT_USB4125-xx-x-0190_6P_TopMnt_Horizontal, symbol Connector:USB_C_Receptacle_PowerOnly_6P
- removed J8: PB, Connector_PinHeader_1.00mm:PinHeader_1x01_P1.00mm_Vertical, symbol Connector:Conn_01x01_Socket
- removed J_BOOST1: U3V70F5_MODULE, Connector_PinHeader_2.54mm:PinHeader_1x04_P2.54mm_Vertical, symbol Connector_Generic:Conn_01x04
- removed Q1: Dual_NMOS_1, Package_TO_SOT_SMD:SOT-23-6, symbol Transistor_FET:Q_Dual_NMOS_S1G1D2S2G2D1
- removed Q2: Q_USB_OR, Package_TO_SOT_SMD:SOT-23, symbol Transistor_FET:Q_PMOS_GDS
- removed Q3: Q_BAT_OR, Package_TO_SOT_SMD:SOT-23, symbol Device:Q_PMOS
- removed Q4: Q_MAIN, Package_TO_SOT_SMD:SOT-23, symbol Transistor_FET:Q_PMOS_GDS
- removed Q5: Q_NMOS_GDS, Package_TO_SOT_SMD:SOT-23, symbol Transistor_FET:Q_NMOS_GDS
- removed R10: 100, Resistor_SMD:R_0805_2012Metric, symbol Device:R_US
- removed R11: 1k, Resistor_SMD:R_0805_2012Metric, symbol Device:R_US
- removed R12, R13, R14: 100k, Resistor_SMD:R_0805_2012Metric, symbol Device:R_Small_US
- removed R18: 100, Resistor_SMD:R_0805_2012Metric, symbol Device:R_Small_US
- removed R19: 10k, Resistor_SMD:R_0805_2012Metric, symbol Device:R_Small_US
- removed R6, R7, R8, R9: 5.1k, Resistor_SMD:R_0805_2012Metric, symbol Device:R_US
- removed U2: MCP73831-2-OT, Package_TO_SOT_SMD:SOT-23-5, symbol Battery_Management:MCP73831-2-OT
- removed U3: DW01A, Package_TO_SOT_SMD:SOT-23-6, symbol Battery_Management:DW01A
- removed U4: AP2112K-3.3, Package_TO_SOT_SMD:SOT-23-5, symbol Regulator_Linear:AP2112K-3.3
- added C28: 470 uF, Capacitor_THT:CP_Radial_D10.0mm_P5.00mm, symbol Device:C_Small
- added C29: 0.1 uF, Capacitor_SMD:C_0805_2012Metric, symbol Device:C_Small
- added C9: 56 nF, Capacitor_SMD:C_0805_2012Metric, symbol Device:C_Small
- added D1, D2: 1N4148, Diode_THT:D_DO-35_SOD27_P7.62mm_Horizontal, symbol Diode:1N4148
- added J10: Lidar, Connector_PinHeader_2.54mm:PinHeader_1x05_P2.54mm_Vertical, symbol Connector_Generic:Conn_01x05
- added J11: J_PI_PWR, Connector_PinHeader_2.54mm:PinHeader_1x04_P2.54mm_Vertical, symbol Connector_Generic:Conn_01x04
- added J12: PIR, Connector_PinSocket_2.54mm:PinSocket_1x02_P2.54mm_Vertical, symbol Connector_Generic:Conn_01x02
- added J15: D24V90F5-A, Connector_PinSocket_2.54mm:PinSocket_1x04_P2.54mm_Vertical, symbol Connector_Generic:Conn_01x04
- added J4: Barrel_Jack, Connector_BarrelJack:BarrelJack_CUI_PJ-102AH_Horizontal, symbol Connector:Barrel_Jack
- added J5: Button Kill Switch, Connector_PinSocket_2.54mm:PinSocket_1x02_P2.54mm_Vertical, symbol Connector_Generic:Conn_01x02
- added J8: D24V90F5-B, Connector_PinSocket_2.54mm:PinSocket_1x04_P2.54mm_Vertical, symbol Connector_Generic:Conn_01x04
- added Q2, Q3: Q_NMOS_GDS, Package_SO:PowerPAK_SO-8_Single, symbol Transistor_FET:Q_NMOS_GDS
- added R8: 49.9k, Resistor_SMD:R_0805_2012Metric, symbol Device:R_Small_US
- added R9: 5.1k, Resistor_SMD:R_0805_2012Metric, symbol Device:R_Small_US
- added TP1: TP ONST1, TestPoint:TestPoint_THTPad_D2.0mm_Drill1.0mm, symbol Connector:TestPoint_Small
- added TP10: TP_M1, TestPoint:TestPoint_THTPad_D2.0mm_Drill1.0mm, symbol Connector:TestPoint
- added TP11: TP_M2, TestPoint:TestPoint_THTPad_D2.0mm_Drill1.0mm, symbol Connector:TestPoint
- added TP12: TP_5V_MAIN, TestPoint:TestPoint_THTPad_D2.0mm_Drill1.0mm, symbol Connector:TestPoint
- added TP13: TP_PWR_KILL, TestPoint:TestPoint_Pad_D1.5mm, symbol Connector:TestPoint
- added TP14: TP_PWR_INT, TestPoint:TestPoint_Pad_D1.5mm, symbol Connector:TestPoint
- added TP15: TP_EN, TestPoint:TestPoint_Pad_D1.5mm, symbol Connector:TestPoint
- added TP16: TP_VCC, TestPoint:TestPoint_THTPad_D2.0mm_Drill1.0mm, symbol Connector:TestPoint
- added TP17: TP_GND3, TestPoint:TestPoint_THTPad_D2.0mm_Drill1.0mm, symbol Connector:TestPoint
- added TP18: TP_GND4, TestPoint:TestPoint_THTPad_D2.0mm_Drill1.0mm, symbol Connector:TestPoint
- added TP19: TP_PCA, TestPoint:TestPoint_THTPad_D2.0mm_Drill1.0mm, symbol Connector:TestPoint
- added TP2: TP ONST2, TestPoint:TestPoint_THTPad_D2.0mm_Drill1.0mm, symbol Connector:TestPoint_Small
- added TP20: TP_SCL, TestPoint:TestPoint_Pad_D1.5mm, symbol Connector:TestPoint
- added TP21: TP_SDA, TestPoint:TestPoint_Pad_D1.5mm, symbol Connector:TestPoint
- added TP4: TP_Jack, TestPoint:TestPoint_THTPad_D2.0mm_Drill1.0mm, symbol Connector:TestPoint
- added TP5: TP_GND1, TestPoint:TestPoint_THTPad_D2.0mm_Drill1.0mm, symbol Connector:TestPoint
- added TP6: TP_PI, TestPoint:TestPoint_THTPad_D2.0mm_Drill1.0mm, symbol Connector:TestPoint
- added TP7: TP_GND2, TestPoint:TestPoint_THTPad_D2.0mm_Drill1.0mm, symbol Connector:TestPoint
- added TP8: TP_5V_SRC, TestPoint:TestPoint_THTPad_D2.0mm_Drill1.0mm, symbol Connector:TestPoint
- added TP9: TP_BAT, TestPoint:TestPoint_THTPad_D2.0mm_Drill1.0mm, symbol Connector:TestPoint
- added U2: TPS2421-2DDAR, Package_SO:SOIC-8-1EP_3.9x4.9mm_P1.27mm_EP2.29x3mm, symbol TPS2421-2:TPS2421-2DDAR
- added U5: LTC4353IMS-PBF, Package_SO:MSOP-16_3x4.039mm_P0.5mm, symbol LTC4353:LTC4353IMS-PBF
- C10, C21: value 0.1 uF -> 47 uF; footprint Capacitor_SMD:C_0805_2012Metric -> Capacitor_SMD:C_1206_3216Metric
- C11: value 22 uF -> 0.1 uF
- C12, C16: footprint Capacitor_SMD:C_0805_2012Metric -> Capacitor_SMD:C_1206_3216Metric
- C14, C17, C24, C25: footprint Capacitor_THT:CP_Radial_D6.3mm_P2.50mm -> Capacitor_THT:CP_Radial_D10.0mm_P5.00mm
- C22: value 47 uF -> 0.1 uF
- C23: value 470 uF -> 47 uF; footprint Capacitor_THT:CP_Radial_D6.3mm_P2.50mm -> Capacitor_SMD:C_1206_3216Metric
- C3: value 22 uF -> 470 uF; footprint Capacitor_SMD:C_0805_2012Metric -> Capacitor_THT:CP_Radial_D10.0mm_P5.00mm
- C5: value 22 uF -> 1 uF
- C6: value 0.1 uF -> 56 nF
- F1: value F_PWR -> 6A-7.5A; footprint Fuse:Fuse_1206_3216Metric -> Fuse:Fuse_2920_7451Metric_Pad2.10x5.45mm_HandSolder
- F3: footprint Fuse:Fuse_1206_3216Metric -> Fuse:Fuse_2920_7451Metric_Pad2.10x5.45mm_HandSolder
- J1: footprint Connector_PinHeader_2.54mm:PinHeader_1x04_P2.54mm_Vertical -> Connector_PinSocket_2.54mm:PinSocket_1x04_P2.54mm_Vertical
- J2, J3: footprint Connector_PinHeader_2.54mm:PinHeader_1x03_P2.54mm_Vertical -> Connector_PinSocket_2.54mm:PinSocket_1x03_P2.54mm_Vertical
- J7: value LTC2954 -> LTC2954-2
- J9: value J_PI_POWER -> Pi GPIO; footprint Connector_PinHeader_1.00mm:PinHeader_1x02_P1.00mm_Vertical -> Connector_PinSocket_2.54mm:PinSocket_1x02_P2.54mm_Vertical
- R16, R17: value 100k -> 10k
Connections:
- net +5V_USB: now also C6.1, D2.2 (A), Q2.3 (S), TP4.1, U5.13 (VIN1)
- net CELL+: now also C10.1, C11.1, J6.2 (Pin_2), J15.1 (Pin_1), J15.2 (Pin_2); no longer C10.2, C11.2, J6.1 (Pin_1)
- net GND: now also C10.2, C11.2, C20.1, C7.2, C8.2, J6.1 (Pin_1), C28.2, C29.2, J10.2 (Pin_2), J11.3 (Pin_3), J11.4 (Pin_4), J12.2 (Pin_2), J15.3 (Pin_3), J15.4 (Pin_4), J4.2, J5.1 (Pin_1), J8.1 (Pin_1), J8.2 (Pin_2), R8.2, TP17.1, TP18.1, TP5.1, TP7.1, U2.4 (GND), U2.EPAD, U5.1 (*EN2), U5.15 (GND), U5.16 (*EN1); no longer C10.1, C11.1, C20.2, C6.2, J9.2 (Pin_2)
- net I2C_SCL: now also J1.4 (Pin_4), J10.4 (Pin_4), TP20.1; no longer J1.3 (Pin_3)
- net I2C_SDA: now also J1.3 (Pin_3), J10.3 (Pin_3), TP21.1; no longer J1.4 (Pin_4)
- net PWR_INT: now also J9.1 (Pin_1), TP14.1
- net PWR_KILL: now also J9.2 (Pin_2), R16.2, TP13.1; no longer R16.1
- net PWR_VBUS_RAW: no longer F1.1
- net SYS_EN: now also TP15.1, U2.2 (*EN)
- net at R5.1, U1.21 (LED14): now also TP10.1
- net at J7.7 (PDT): now also C20.2; no longer C20.1
- net at J7.2 (PB): now also C8.1, R9.2
- net at R4.1, U1.22 (LED15): now also TP11.1
- net 3V3 renamed +3.3V_PI
- net +3.3V_PI: now also R16.1, J10.5 (Pin_5), J12.1 (Pin_1), TP19.1, TP6.1
- net 5V_BAT renamed +5V_BAT
- net +5V_BAT: now also C21.1, C29.1, C9.2, D1.2 (A), J8.3 (Pin_3), J8.4 (Pin_4), Q3.3 (S), TP9.1, U5.4 (VIN2)
- net 5V_MAIN renamed +5V_MAIN
- net +5V_MAIN: now also C28.1, J10.1 (Pin_1), TP12.1, U2.7 (VOUT); no longer C21.1
- net 5V_PI: no longer names the net of F3.2
- net 5V_PI: now also J11.1 (Pin_1), J11.2 (Pin_2); no longer J9.1 (Pin_1)
- net 5V_SRC renamed +5V_SRC
- net +5V_SRC: now also Q2.2 (D), Q3.2 (D), TP8.1, U2.3 (VIN), U5.10 (OUT1), U5.7 (OUT2); no longer R16.2
- removed net CELL-: C7.2, C8.1, J6.2 (Pin_2)
- net CHG_VBUS: no longer names the net of C5.1
- net CHG_VBUS: now also U2.6 (CT); no longer C6.1
- new net: R8.1, U2.5 (ISET)
- new net: D1.1 (K), D2.1 (K), TP16.1, U5.14 (VCC)
- new net: Q3.1 (G), U5.5 (GATE2)
- new net: J5.2 (Pin_2), R9.1
- new net: C6.2, U5.11 (CPO1)
- new net: F1.1, J4.1
- new net: Q2.1 (G), U5.12 (GATE1)
- new net: C9.1, U5.6 (CPO2)
- new net: TP2.1, U5.8 (*ONST2)
- new net: TP1.1, U5.9 (*ONST1)
- no-connect marks 16 -> 17
Other:
- note added: "Barrel Jack"
- note added: "To GPIO pins for PWR_KILL and PWR_INT"
- note removed: "5V to 3.3V LDO"
- note removed: "5V_MAIN from 5V_SOURCE"
- note removed: "Battery Charging IC and Protection Circuit"
- note removed: "Boost Converter"
- note removed: "OR Gate - 5V_USB & 5V_BAT"
- note removed: "USB-C Charging"
- note removed: "USB-C Power"
- moved on the sheet: C12, C13, C14, C15, C16, C17, C18, C19, C20, C3, C4, C7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
